Commit message: 0612:compile repo on nx

File: src/zed-ros-wrapper/zed_wrapper/urdf/zed_descr.urdf.xacro (robot description, xacro)
@@ -16,17 +16,100 @@
 -->
 <robot name="stereolabs_camera" xmlns:xacro="http://ros.org/wiki/xacro">
-  <xacro:arg name="camera_name"   default="zed" />
-  <xacro:arg name="camera_model"  default="zed" />
-  <xacro:arg name="base_frame"    default="base_link" />
-  <xacro:arg name="cam_pos_x"     default="0.0" />
-  <xacro:arg name="cam_pos_y"     default="0.0" />
-  <xacro:arg name="cam_pos_z"     default="0.0" />
-  <xacro:arg name="cam_roll"      default="0.0" />
-  <xacro:arg name="cam_pitch"     default="0.0" />
-  <xacro:arg name="cam_yaw"       default="0.0" />
-  <xacro:include filename="$(find zed_wrapper)/urdf/zed_macro.urdf.xacro" />
-  <xacro:zed_camera name="$(arg camera_name)" model="$(arg camera_model)" parent="$(arg base_frame)">
-    <origin xyz="$(arg cam_pos_x) $(arg cam_pos_y) $(arg cam_pos_z)" rpy="$(arg cam_roll) $(arg cam_pitch) $(arg cam_yaw)" />
-  </xacro:zed_camera>
-  <link name="$(arg base_frame)" />
+<!-- Includes -->
+    <xacro:include filename="$(find zed_wrapper)/urdf/include/materials.urdf.xacro" />
+    <!-- Arguments -->
+    <xacro:arg name="camera_name"   default="zed" />
+    <xacro:arg name="camera_model"  default="zed" />
+    <xacro:arg name="base_frame"    default="base_link" />
+    <xacro:arg name="cam_pos_x"     default="0.0" />
+    <xacro:arg name="cam_pos_y"     default="0.0" />
+    <xacro:arg name="cam_pos_z"     default="0.0" />
+    <xacro:arg name="cam_roll"      default="0.0" />
+    <xacro:arg name="cam_pitch"     default="0.0" />
+    <xacro:arg name="cam_yaw"       default="0.0" />
+    <!-- Properties -->
+    <xacro:property name="M_PI"     value="3.1415926535897931" />
+    <xacro:property name="model"    value="$(arg camera_model)" />
+    <xacro:if value="${model == 'zed'}">
+        <xacro:property name="baseline" value="0.12" />
+    </xacro:if>
+    <xacro:if value="${model == 'zedm'}">
+        <xacro:property name="baseline" value="0.06" />
+    </xacro:if>
+    <xacro:if value="${model == 'zed2'}">
+        <xacro:property name="baseline" value="0.12" />
+    </xacro:if>
+    <xacro:if value="${model == 'zed2i'}">
+        <xacro:property name="baseline" value="0.12" />
+    </xacro:if>
+<!-- base_link -->
+    <link name="$(arg base_frame)" />
+<!-- Camera Center -->
+    <joint name="$(arg camera_name)_camera_center_joint" type="fixed">
+        <parent link="$(arg base_frame)"/>
+        <child link="$(arg camera_name)_camera_center"/>
+        <origin xyz="$(arg cam_pos_x) $(arg cam_pos_y) $(arg cam_pos_z)" rpy="$(arg cam_roll) $(arg cam_pitch) $(arg cam_yaw)" />
+    </joint>
+    <link name="$(arg camera_name)_camera_center">
+        <visual>
+            <origin xyz="0 0 0" rpy="0 0 0"/>
+            <geometry>
+                <mesh filename="package://zed_wrapper/urdf/models/${model}.stl" />
+            </geometry>
+            <material name="${model}_mat" />
+        </visual>
+    </link>
+<!-- Left Camera -->
+    <joint name="$(arg camera_name)_left_camera_joint" type="fixed">
+        <parent link="$(arg camera_name)_camera_center"/>
+        <child link="$(arg camera_name)_left_camera_frame"/>
+        <origin xyz="0 ${baseline/2} 0" rpy="0 0 0" />
+    </joint>
+    <link name="$(arg camera_name)_left_camera_frame" />
+    <joint name="$(arg camera_name)_left_camera_optical_joint" type="fixed">
+        <origin xyz="0 0 0" rpy="-${M_PI/2} 0.0 -${M_PI/2}"/>
+        <parent link="$(arg camera_name)_left_camera_frame"/>
+        <child link="$(arg camera_name)_left_camera_optical_frame"/>
+    </joint>
+    <link name="$(arg camera_name)_left_camera_optical_frame"/>
+<!-- Right Camera -->
+    <joint name="$(arg camera_name)_right_camera_joint" type="fixed">
+        <parent link="$(arg camera_name)_camera_center"/>
+        <child link="$(arg camera_name)_right_camera_frame"/>
+        <origin xyz="0 -${baseline/2} 0" rpy="0 0 0" />
+    </joint>
+    <link name="$(arg camera_name)_right_camera_frame" />
+    <joint name="$(arg camera_name)_right_camera_optical_joint" type="fixed">
+        <origin xyz="0 0 0" rpy="-${M_PI/2} 0.0 -${M_PI/2}"/>
+        <parent link="$(arg camera_name)_right_camera_frame"/>
+        <child link="$(arg camera_name)_right_camera_optical_frame"/>
+    </joint>
+    <link name="$(arg camera_name)_right_camera_optical_frame"/>
+<!-- ZED2 Sensors -->
+    <xacro:if value="${model == 'zed2'}">
+        <joint name="$(arg camera_name)_mag_joint" type="fixed">
+            <parent link="$(arg camera_name)_camera_center"/>
+            <child link="$(arg camera_name)_mag_link"/>
+            <origin xyz="0 0 0" rpy="0 0 0" />
+        </joint>
+        <link name="$(arg camera_name)_mag_link" />
+        <joint name="$(arg camera_name)_baro_joint" type="fixed">
+            <parent link="$(arg camera_name)_camera_center"/>
+            <child link="$(arg camera_name)_baro_link"/>
+            <origin xyz="0 0 0" rpy="0 0 0" />
+        </joint>
+        <link name="$(arg camera_name)_baro_link" />
+        <joint name="$(arg camera_name)_temp_left_joint" type="fixed">
+            <parent link="$(arg camera_name)_left_camera_frame"/>
+            <child link="$(arg camera_name)_temp_left_link"/>
+            <origin xyz="0 0 0" rpy="0 0 0" />
+        </joint>
+        <link name="$(arg camera_name)_temp_left_link" />
+        <joint name="$(arg camera_name)_temp_right_joint" type="fixed">
+            <parent link="$(arg camera_name)_right_camera_frame"/>
+            <child link="$(arg camera_name)_temp_right_link"/>
+            <origin xyz="0 0 0" rpy="0 0 0" />
+        </joint>
+        <link name="$(arg camera_name)_temp_right_link" />
+    </xacro:if>
 </robot>
